File: cccamp2019_xil_badge.kicad_pcb (KiCad board)
At the start: 2 copper layers, 62.8 x 46.5 mm, 0 parts

Commit message: More work
Parts:
- added BT1: Battery_Cell, Battery_Extra:CR1632, B.Cu at (144.1, 109.4)
- added C1: 0.1uF, Capacitor_SMD:C_0603_1608Metric, B.Cu at (170.8, 101.4)
- added D1: LED_RGBA, LED_SMD_Extra:LED_RGBA_0606_UpsideDown, B.Cu at (154.5, 80.4)
- added D2: LED_RGBA, LED_SMD_Extra:LED_RGBA_0606_UpsideDown, B.Cu at (161.5, 89.0)
- added D4: LED_RGBA, LED_SMD_Extra:LED_RGBA_0606_UpsideDown, B.Cu at (126.5, 89.0)
- added D5: LED_RGBA, LED_SMD_Extra:LED_RGBA_0606_UpsideDown, B.Cu at (133.5, 80.4)
- added Q1: BSS84, Package_TO_SOT_SMD:SOT-23, B.Cu at (116.9, 98.1)
- added R1: TBD, Resistor_SMD:R_0603_1608Metric, B.Cu at (173.5, 95.3)
- added R2: TBD, Resistor_SMD:R_0603_1608Metric, B.Cu at (171.7, 95.3)
- added R3: TBD, Resistor_SMD:R_0603_1608Metric, B.Cu at (169.9, 95.3)
- added R7: 1K, Resistor_SMD:R_0603_1608Metric, B.Cu at (166.6, 110.9)
- added REF**: Safety_Pin_45mm, Socket_Extra:Safety_Pin_45mm, B.Cu at (144.3, 97.9)
- added SW1: SW_SPDT, Button_Switch_SMD:SW_SPDT_PCM12, B.Cu at (160.5, 111.5)
- added TP1: TP_SWDIO, TestPoint:TestPoint_Pad_D1.0mm, B.Cu at (158.3, 104.5)
- added TP2: TP_GND, TestPoint:TestPoint_Pad_D1.0mm, B.Cu at (156.5, 104.5)
- added TP3: TP_SWCLK, TestPoint:TestPoint_Pad_D1.0mm, B.Cu at (154.7, 104.5)
- added TP4: TP_VDD, TestPoint:TestPoint_Pad_D1.0mm, B.Cu at (152.9, 104.5)
- added U1: ATSAMD09C13A, Package_SO:SOIC-14_3.9x8.7mm_P1.27mm, B.Cu at (169.4, 105.9)
Routing:
- net VDD: track 0.00 -> 93.7 mm
- net /ANODE1: track 0.00 -> 75.9 mm, vias 0 -> 2
- net Net-(D1-Pad3): track 0.00 -> 66.3 mm
- net Net-(D1-Pad4): track 0.00 -> 63.1 mm
- net Net-(D1-Pad2): track 0.00 -> 61.4 mm
- net Net-(D1-Pad1): track 0.00 -> 60.5 mm
- net GND: track 0.00 -> 33.0 mm
- net /SWCLK: track 0.00 -> 17.0 mm
- net /BLUE1: track 0.00 -> 13.5 mm
- net /RED1: track 0.00 -> 8.84 mm
- net /SWDIO: track 0.00 -> 8.08 mm
- net /GREEN1: track 0.00 -> 7.96 mm
- net +BATT: track 0.00 -> 7.44 mm
Other:
- outline, holes or cut-outs redrawn
- net class Default: clearance 0.2 -> 0.15; trace_width 0.25 -> 0.15; via_dia 0.8 -> 0.55; via_drill 0.4 -> 0.3
- rule solder_mask_min_width: 0.25 -> 0.15
- rule trace_clearance: 0.2 -> 0.15
- rule trace_min: 0.2 -> 0.15
- rule via_min_size: 0.4 -> 0.55
- board text added: "3.3"
- board text added: "CLK"
- board text added: "GND"
- board text added: "IO"
- board text added: "JLCJLCJLCJLC"
