File: cccamp2019_xil_badge.sch (KiCad schematic (older format))
At the start: 1 part

Commit message: More work
Parts:
- added BT1: Battery_Cell, Battery_Extra:CR1632, symbol Device:Battery_Cell
- added C1: 0.1uF, Capacitor_SMD:C_0603_1608Metric, symbol Device:C_Small
- added D1, D2, D4, D5: LED_RGBA, LED_SMD_Extra:LED_RGBA_0606_UpsideDown, symbol Device:LED_RGBA
- added Q1: BSS84, Package_TO_SOT_SMD:SOT-23, symbol Transistor_FET:BSS84
- added R1, R2, R3: TBD, Resistor_SMD:R_0603_1608Metric, symbol Device:R_Small
- added R7: 1K, Resistor_SMD:R_0603_1608Metric, symbol Device:R_Small
- added SW1: SW_SPDT, Button_Switch_SMD:SW_SPDT_PCM12, symbol Switch:SW_SPDT
- added TP1: TP_SWDIO, TestPoint:TestPoint_Pad_D1.0mm, symbol Connector:TestPoint
- added TP2: TP_GND, TestPoint:TestPoint_Pad_D1.0mm, symbol Connector:TestPoint
- added TP3: TP_SWCLK, TestPoint:TestPoint_Pad_D1.0mm, symbol Connector:TestPoint
- added TP4: TP_VDD, TestPoint:TestPoint_Pad_D1.0mm, symbol Connector:TestPoint
- gave numbers to parts that had none: 1
Connections:
- net labels added: +BATT, ANODE1, BLUE1, GND, GREEN1, RED1, SWCLK, SWDIO, VDD
- wire segments 0 -> 70
- no-connect marks 0 -> 2
Other:
- moved on the sheet: U1
